File: _autosave-weiland-esp32.kicad_sch (KiCad schematic)
At the start: 19 parts, among them J1 Conn_01x04_Pin, J3 Conn_01x04_Pin, J5 Conn_02x03_Odd_Even, U1 ESP32-WROOM-32E(8MB), U2 AMS1117-3.3_C347222, U3 GR6205-SOP-8, U4 MAX98357AEWL_T

Commit message: antenna can't be on the board itself (interference)
Parts:
- J5: footprint (none) -> Connector_PinSocket_1.27mm:PinSocket_2x03_P1.27mm_Vertical_SMD
Changed lines of the file:
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@@
 			)
 		)
-		(property "Footprint" ""
+		(property "Footprint" "Connector_PinSocket_1.27mm:PinSocket_2x03_P1.27mm_Vertical_SMD"
 			(at 104.14 30.48 0)
 			(effects
