File: _autosave-weiland-esp32.kicad_pcb (KiCad board)
At the start: 2 copper layers, 20.2 x 58 mm, 22 parts, among them J1 S02B-PASK-2, J2 20021221-00006T4LF, J3 S02B-PASK-2, J4 S02B-PASK-2, J6 S02B-PASK-2, J7 S02B-PASK-2, U1 ESP32-WROOM-32E(8MB), U2 AMS1117-3.3_C347222, U3 GR6205-SOP-8, U4 MAX98357AEWL_T

Commit message: jst connectors
Parts:
- moved J4 1.40 mm to (129.9, 78.9)
- moved J7 1.10 mm to (143.2, 78.9)
- moved J1 0.21 mm to (145.2, 119.7)
- moved J3 0.12 mm to (138.5, 119.7)
Changed lines of the file:
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@@
 	(footprint "footprints:CONN2_S02B-PASK-2_JST"
 		(layer "F.Cu")
-		(at 131.299999 78.9)
+		(at 129.899999 78.9)
 		(tags "S02B-PASK-2 ")
 		(property "Reference" "J4"
@@
 	(footprint "footprints:CONN2_S02B-PASK-2_JST"
 		(layer "F.Cu")
-		(at 145.399999 119.6 180)
+		(at 145.1951 119.654699 180)
 		(tags "S02B-PASK-2 ")
 		(property "Reference" "J1"
@@
 	(footprint "footprints:CONN2_S02B-PASK-2_JST"
 		(layer "F.Cu")
-		(at 142.099999 78.9)
+		(at 143.199999 78.9)
 		(tags "S02B-PASK-2 ")
 		(property "Reference" "J7"
@@
 	(footprint "footprints:CONN2_S02B-PASK-2_JST"
 		(layer "F.Cu")
-		(at 138.6 119.6 180)
+		(at 138.4951 119.654699 180)
 		(tags "S02B-PASK-2 ")
 		(property "Reference" "J3"
