File: weiland-esp32.kicad_sch (KiCad schematic)
At the start: 36 parts, among them J1 S02B-PASK-2, J6 S02B-PASK-2, J7 S02B-PASK-2, P1 S04B-PASK-2_LF__SN_, P2 S04B-PASK-2_LF__SN_, U1 ESP32-WROOM-32E(8MB), U2 AMS1117-3.3_C347222, U3 MAX98357AETE_T, U5 ULN2003F12FN-7, U6 DZ127S-22-06-55

Commit message: board complete
Parts:
- added H3, H4: MountingHole, MountingHole:MountingHole_3.2mm_M3, symbol Mechanical:MountingHole
- renumbered IO14 to I14, IO15 to I15, IO16 to I16, IO17 to I17, IO18 to I18, IO19 to I19, IO22 to I22, OUTN1 to N1, OUTP1 to P+1, 3.3V1 to V3
Connections:
- net OUTA: now also P2.4; no longer P2.2
- net OUTB: now also P2.2; no longer P2.4
Changed lines of the file:
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@@
 		)
 	)
-	(label "OUTB"
-		(at 77.47 66.04 180)
+	(label "IO0"
+		(at 96.52 158.75 0)
 		(fields_autoplaced yes)
 		(effects
@@
 				(size 1.27 1.27)
 			)
-			(justify right bottom)
+			(justify left)
 		)
 	)
-	(label "IO0"
-		(at 96.52 158.75 0)
+	(label "EN"
+		(at 12.7 147.32 0)
 		(fields_autoplaced yes)
 		(effects
@@
 				(size 1.27 1.27)
 			)
-			(justify left)
+			(justify left bottom)
 		)
 	)
-	(label "EN"
-		(at 12.7 147.32 0)
+	(label "OUTA"
+		(at 77.47 66.04 180)
 		(fields_autoplaced yes)
 		(effects
@@
 				(size 1.27 1.27)
 			)
-			(justify left bottom)
+			(justify right bottom)
 		)
 	)
@@
 		)
 	)
-	(label "OUTA"
+	(label "OUTB"
 		(at 77.47 60.96 180)
 		(fields_autoplaced yes)
@@
 		(dnp no)
 		(fields_autoplaced yes)
-		(property "Reference" "IO19"
+		(property "Reference" "I19"
 			(at 341.63 133.8579 0)
 			(effects
@@
 			(project "weiland-esp32"
 				(path "/745a8d65-fa51-45f7-9665-7610e72f2a80"
-					(reference "IO19")
+					(reference "I19")
 					(unit 1)
 				)
@@
 		(dnp no)
 		(fields_autoplaced yes)
-		(property "Reference" "IO22"
+		(property "Reference" "I22"
 			(at 356.87 146.5579 0)
 			(effects
@@
 			(project "weiland-esp32"
 				(path "/745a8d65-fa51-45f7-9665-7610e72f2a80"
-					(reference "IO22")
+					(reference "I22")
 					(unit 1)
 				)
@@
 	)
 	(symbol
+		(lib_id "Mechanical:MountingHole")
+		(at 372.11 194.31 0)
+		(unit 1)
+		(exclude_from_sim yes)
+		(in_bom no)
+		(on_board yes)
+		(dnp no)
+		(fields_autoplaced yes)
+		(property "Reference" "H4"
+			(at 374.65 193.0399 0)
+			(effects
+				(font
+					(size 1.27 1.27)
+				)
+				(justify left)
+			)
+		)
+		(property "Value" "MountingHole"
+			(at 374.65 195.5799 0)
+			(effects
+				(font
+					(size 1.27 1.27)
+				)
+				(justify left)
+			)
+		)
+		(property "Footprint" "MountingHole:MountingHole_3.2mm_M3"
+			(at 372.11 194.31 0)
+			(effects
+				(font
+					(size 1.27 1.27)
+				)
+				(hide yes)
+			)
+		)
+		(property "Datasheet" "~"
+			(at 372.11 194.31 0)
+			(effects
+				(font
+					(size 1.27 1.27)
+				)
+				(hide yes)
+			)
+		)
+		(property "Description" "Mounting Hole without connection"
+			(at 372.11 194.31 0)
+			(effects
+				(font
+					(size 1.27 1.27)
+				)
+				(hide yes)
+			)
+		)
+		(instances
+			(project "weiland-esp32"
+				(path "/745a8d65-fa51-45f7-9665-7610e72f2a80"
+					(reference "H4")
+					(unit 1)
+				)
+			)
+		)
+	)
+	(symbol
 		(lib_id "Device:C")
 		(at 290.83 53.34 90)
@@
 		(dnp no)
 		(fields_autoplaced yes)
-		(property "Reference" "IO16"
+		(property "Reference" "I16"
 			(at 386.08 133.8579 0)
 			(effects
@@
 			(project "weiland-esp32"
 				(path "/745a8d65-fa51-45f7-9665-7610e72f2a80"
-					(reference "IO16")
+					(reference "I16")
 					(unit 1)
 				)
@@
 		(dnp no)
 		(fields_autoplaced yes)
-		(property "Reference" "IO18"
+		(property "Reference" "I18"
 			(at 355.6 133.8579 0)
 			(effects
@@
 			(project "weiland-esp32"
 				(path "/745a8d65-fa51-45f7-9665-7610e72f2a80"
-					(reference "IO18")
+					(reference "I18")
 					(unit 1)
 				)
@@
 		(dnp no)
 		(fields_autoplaced yes)
-		(property "Reference" "IO17"
+		(property "Reference" "I17"
 			(at 370.84 133.8579 0)
 			(effects
@@
 			(project "weiland-esp32"
 				(path "/745a8d65-fa51-45f7-9665-7610e72f2a80"
-					(reference "IO17")
+					(reference "I17")
 					(unit 1)
 				)
@@
 		(dnp no)
 		(fields_autoplaced yes)
-		(property "Reference" "3.3V1"
+		(property "Reference" "V3"
 			(at 341.63 121.1579 0)
 			(effects
@@
 			(project ""
 				(path "/745a8d65-fa51-45f7-9665-7610e72f2a80"
-					(reference "3.3V1")
+					(reference "V3")
 					(unit 1)
 				)
@@
 		(dnp no)
 		(fields_autoplaced yes)
-		(property "Reference" "IO14"
+		(property "Reference" "I14"
 			(at 370.84 146.5579 0)
 			(effects
@@
 			(project "weiland-esp32"
 				(path "/745a8d65-fa51-45f7-9665-7610e72f2a80"
-					(reference "IO14")
+					(reference "I14")
 					(unit 1)
 				)
@@
 		(dnp no)
 		(fields_autoplaced yes)
-		(property "Reference" "OUTN1"
+		(property "Reference" "N1"
 			(at 356.87 159.2579 0)
 			(effects
@@
 			(project "weiland-esp32"
 				(path "/745a8d65-fa51-45f7-9665-7610e72f2a80"
-					(reference "OUTN1")
+					(reference "N1")
 					(unit 1)
 				)
@@
 		(dnp no)
 		(fields_autoplaced yes)
-		(property "Reference" "IO15"
+		(property "Reference" "I15"
 			(at 341.63 146.5579 0)
 			(effects
@@
 			(project "weiland-esp32"
 				(path "/745a8d65-fa51-45f7-9665-7610e72f2a80"
-					(reference "IO15")
+					(reference "I15")
 					(unit 1)
 				)
@@
 	)
 	(symbol
+		(lib_id "Mechanical:MountingHole")
+		(at 372.11 187.96 0)
+		(unit 1)
+		(exclude_from_sim yes)
+		(in_bom no)
+		(on_board yes)
+		(dnp no)
+		(fields_autoplaced yes)
+		(property "Reference" "H3"
+			(at 374.65 186.6899 0)
+			(effects
+				(font
+					(size 1.27 1.27)
+				)
+				(justify left)
+			)
+		)
+		(property "Value" "MountingHole"
+			(at 374.65 189.2299 0)
+			(effects
+				(font
+					(size 1.27 1.27)
+				)
+				(justify left)
+			)
+		)
+		(property "Footprint" "MountingHole:MountingHole_3.2mm_M3"
+			(at 372.11 187.96 0)
+			(effects
+				(font
+					(size 1.27 1.27)
+				)
+				(hide yes)
+			)
+		)
+		(property "Datasheet" "~"
+			(at 372.11 187.96 0)
+			(effects
+				(font
+					(size 1.27 1.27)
+				)
+				(hide yes)
+			)
+		)
+		(property "Description" "Mounting Hole without connection"
+			(at 372.11 187.96 0)
+			(effects
+				(font
+					(size 1.27 1.27)
+				)
+				(hide yes)
+			)
+		)
+		(instances
+			(project "weiland-esp32"
+				(path "/745a8d65-fa51-45f7-9665-7610e72f2a80"
+					(reference "H3")
+					(unit 1)
+				)
+			)
+		)
+	)
+	(symbol
 		(lib_id "CL05B104KO5NNNC_1")
 		(at 38.1 134.62 0)
@@
 		(dnp no)
 		(fields_autoplaced yes)
-		(property "Reference" "OUTP1"
+		(property "Reference" "P+1"
 			(at 341.63 159.2579 0)
 			(effects
@@
 			(project "weiland-esp32"
 				(path "/745a8d65-fa51-45f7-9665-7610e72f2a80"
-					(reference "OUTP1")
+					(reference "P+1")
 					(unit 1)
 				)
